File: hardware/mainboard/mainboard.kicad_sch (KiCad schematic)
At the start: 52 parts, among them J1 USB-C, J2 4.3" RGB panel, J3 GT911 touch, J4 SparkFun 2D Barcode Scanner, J5 UART scanner (GM65), J6 LD2410C radar, Q1 AO3400A, SW1 RESET, SW2 BOOT, U1 USBLC6-2SC6, U2 SY8089AAAC, U3 ESP32-S3-WROOM-1-N16R8, U4 74AHCT1G125, U5 TPS61169

Commit message: Drop the presence radar
A scan already wakes the screen, so the LD2410C radar only saved a glance at
the dim clock. Gone from:

- firmware: pantry-feedback.yaml no longer has the presence sensor; the
  carrier package loses the radar UART and ld2410
- scanner carrier: the 5-pin radar header, its three resistors and the
  Sunton P2 connector it needed (two cables to the Sunton now, not three)
- mainboard: the radar header and its resistor; IO4 is free
- enclosure: the radar rails; the chin shrinks to 15 mm, so the case is
  now 111 x 139 x 51 mm

Both boards rebuilt clean (ERC 0, DRC 0 / 0 unconnected / 0 footprint
errors). On the mainboard the ribbon connector is now the only part whose
fine-pitch ground pins rely on the pour; U5's narrow ground pin gets a via
again. All four firmware configs validate.
Parts:
- removed J6: LD2410C radar, Connector_PinHeader_2.54mm:PinHeader_1x03_P2.54mm_Vertical, symbol Connector_Generic:Conn_01x03
- removed R20: 1k, Resistor_SMD:R_0603_1608Metric, symbol Device:R
Connections:
- net PRESENCE: no longer names the net of U3.4 (IO4)
- no-connect marks 11 -> 12
Other:
- note removed: "Radar: HLK-LD2410C OUT -> IO4 (wakes the screen)."
Changed lines of the file:
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@@
 		)
 	)
-	(label "PRESENCE"
-		(at 185.42 101.6 180)
-		(fields_autoplaced yes)
-		(effects
-			(font
-				(size 1.27 1.27)
-			)
-			(justify right bottom)
-		)
+	(no_connect
+		(at 185.42 101.6)
 	)
 	(label "BL_PWM"
@@
 	)
 	(symbol
-		(lib_id "Connector_Generic:Conn_01x03")
-		(at 30.48 83.82 0)
-		(unit 1)
-		(exclude_from_sim no)
-		(in_bom yes)
-		(on_board yes)
-		(dnp no)
-		(property "Reference" "J6"
-			(at 30.48 78.74 0)
-			(effects
-				(font
-					(size 1.27 1.27)
-				)
-			)
-		)
-		(property "Value" "LD2410C radar"
-			(at 30.48 88.9 0)
-			(effects
-				(font
-					(size 1.27 1.27)
-				)
-			)
-		)
-		(property "Footprint" "Connector_PinHeader_2.54mm:PinHeader_1x03_P2.54mm_Vertical"
-			(at 30.48 83.82 0)
-			(hide yes)
-			(effects
-				(font
-					(size 1.27 1.27)
-				)
-			)
-		)
-		(property "Datasheet" ""
-			(at 30.48 83.82 0)
-			(hide yes)
-			(effects
-				(font
-					(size 1.27 1.27)
-				)
-			)
-		)
-		(property "Description" "Generic connector, single row, 01x03, script generated (kicad-library-utils/schlib/autogen/connector/)"
-			(at 30.48 83.82 0)
-			(hide yes)
-			(effects
-				(font
-					(size 1.27 1.27)
-				)
-			)
-		)
-		(property "LCSC" "C2937625"
-			(at 30.48 83.82 0)
-			(hide yes)
-			(effects
-				(font
-					(size 1.27 1.27)
-				)
-			)
-		)
-		(property "Pins" "1 5V / 2 GND / 3 OUT"
-			(at 30.48 83.82 0)
-			(hide yes)
-			(effects
-				(font
-					(size 1.27 1.27)
-				)
-			)
-		)
-		(pin "1"
-		)
-		(pin "2"
-		)
-		(pin "3"
-		)
-		(instances
-			(project "mainboard"
-				(path "/1485f497-d9c3-5dfb-b6bd-ebc7ec208940"
-					(reference "J6")
-					(unit 1)
-				)
-			)
-		)
-	)
-	(label "+5V"
-		(at 25.4 81.28 180)
-		(fields_autoplaced yes)
-		(effects
-			(font
-				(size 1.27 1.27)
-			)
-			(justify right bottom)
-		)
-	)
-	(label "GND"
-		(at 25.4 83.82 180)
-		(fields_autoplaced yes)
-		(effects
-			(font
-				(size 1.27 1.27)
-			)
-			(justify right bottom)
-		)
-	)
-	(label "RADAR_OUT"
-		(at 25.4 86.36 180)
-		(fields_autoplaced yes)
-		(effects
-			(font
-				(size 1.27 1.27)
-			)
-			(justify right bottom)
-		)
-	)
-	(symbol
-		(lib_id "Device:R")
-		(at 55.88 83.82 0)
-		(unit 1)
-		(exclude_from_sim no)
-		(in_bom yes)
-		(on_board yes)
-		(dnp no)
-		(property "Reference" "R20"
-			(at 57.912 83.82 0)
-			(effects
-				(font
-					(size 1.27 1.27)
-				)
-			)
-		)
-		(property "Value" "1k"
-			(at 55.88 83.82 0)
-			(effects
-				(font
-					(size 1.27 1.27)
-				)
-			)
-		)
-		(property "Footprint" "Resistor_SMD:R_0603_1608Metric"
-			(at 54.102 83.82 0)
-			(hide yes)
-			(effects
-				(font
-					(size 1.27 1.27)
-				)
-			)
-		)
-		(property "Datasheet" ""
-			(at 55.88 83.82 0)
-			(hide yes)
-			(effects
-				(font
-					(size 1.27 1.27)
-				)
-			)
-		)
-		(property "Description" "Resistor"
-			(at 55.88 83.82 0)
-			(hide yes)
-			(effects
-				(font
-					(size 1.27 1.27)
-				)
-			)
-		)
-		(property "LCSC" "C21190"
-			(at 55.88 83.82 0)
-			(hide yes)
-			(effects
-				(font
-					(size 1.27 1.27)
-				)
-			)
-		)
-		(pin "1"
-		)
-		(pin "2"
-		)
-		(instances
-			(project "mainboard"
-				(path "/1485f497-d9c3-5dfb-b6bd-ebc7ec208940"
-					(reference "R20")
-					(unit 1)
-				)
-			)
-		)
-	)
-	(label "RADAR_OUT"
-		(at 55.88 80.01 90)
-		(fields_autoplaced yes)
-		(effects
-			(font
-				(size 1.27 1.27)
-			)
-			(justify left bottom)
-		)
-	)
-	(label "PRESENCE"
-		(at 55.88 87.63 270)
-		(fields_autoplaced yes)
-		(effects
-			(font
-				(size 1.27 1.27)
-			)
-			(justify right bottom)
-		)
-	)
-	(symbol
 		(lib_id "Mechanical:MountingHole")
 		(at 200.66 190.5 0)
@@
 		(effects
 			(font
-				(size 1.27 1.27)
-			)
-			(justify left bottom)
-		)
-	)
-	(text "Radar: HLK-LD2410C OUT -> IO4 (wakes the screen)."
-		(exclude_from_sim no)
-		(at 15 75 0)
-		(effects
-			(font
