File: hardware/scanner-carrier/scanner-carrier.kicad_pcb (KiCad board)
At the start: 2 copper layers, 64 x 44 mm, 31 parts, among them J1 Sunton P1 UART, J2 Sunton P4 IO, J3 SparkFun 2D Barcode Scanner, J4 GM65 scanner, J5 LD2410C radar, J6 Sunton P2 IO, Q1 AO3400A, U1 AMS1117-3.3, U2 74AHCT1G125

Commit message: Scanner carrier: fix overlapping parts, share the feedback package
The KiCad project defaults came from a demo that ignores courtyard overlaps,
so DRC never checked them. With the check on, six pairs overlapped: the
buzzer, radar header, LED, a corner hole and a test pad are moved apart, and
the second SparkFun standoff (H2) is gone: its hole is 4 mm from the
header's GND pin, so a standoff can't sit next to the socket there. DRC is
clean again with the check on.

Firmware: the buzzer, status LED, presence sensor and the scan feedback
script move to pantry-feedback.yaml, which takes its pins as vars, so the
carrier and the new mainboard share it. The carrier package keeps its radar
UART. The LED uses channel_colors (rgb_order is deprecated).
Parts:
- removed H2: M3 standoff (scanner), MountingHole:MountingHole_3.2mm_M3
- moved H4 11.0 mm to (160.5, 120.5)
- moved TP3 2.82 mm to (159.8, 113.5)
- moved D1 1.58 mm to (146.0, 96.0)
- moved LS1 1.41 mm to (152.0, 104.5)
Routing:
- net /LED_3V3: track 30.1 -> 34.3 mm
- net /+5V: track 104.9 -> 108.3 mm, vias 6 -> 4
- net /SCAN_RX: track 53.5 -> 55.3 mm, vias 3 -> 4
- net /IO13_RXD: track 33.6 -> 34.9 mm, vias 0 -> 2
- net /LED_DIN: track 28.5 -> 29.8 mm
- net /LED_DOUT: track 5.66 -> 6.81 mm
- net /SCAN_TX: track 56.8 -> 55.8 mm, vias 0 -> 3
- net /IO11_TXD: track 30.5 -> 29.5 mm
- net /BUZZ_SW: track 15.8 -> 15.5 mm, vias 2 -> 0
- net /IO12_PRESENCE: track 39.9 -> 40.1 mm, vias 4 -> 6
- net /RADAR_TX: track 5.84 -> 5.73 mm, vias 1 -> 0
- net /SCAN_TRIG: vias 1 -> 0
- net /SCAN_STAT: vias 1 -> 0
Other:
- board text added: "SparkFun 2D Barcode Scanner (11 mm standoff in H1)"
- board text removed: "SparkFun 2D Barcode Scanner (on 11 mm standoffs)"

Commit message: Drop the presence radar
A scan already wakes the screen, so the LD2410C radar only saved a glance at
the dim clock. Gone from:

- firmware: pantry-feedback.yaml no longer has the presence sensor; the
  carrier package loses the radar UART and ld2410
- scanner carrier: the 5-pin radar header, its three resistors and the
  Sunton P2 connector it needed (two cables to the Sunton now, not three)
- mainboard: the radar header and its resistor; IO4 is free
- enclosure: the radar rails; the chin shrinks to 15 mm, so the case is
  now 111 x 139 x 51 mm

Both boards rebuilt clean (ERC 0, DRC 0 / 0 unconnected / 0 footprint
errors). On the mainboard the ribbon connector is now the only part whose
fine-pitch ground pins rely on the pour; U5's narrow ground pin gets a via
again. All four firmware configs validate.
Parts:
- removed J5: LD2410C radar, Connector_PinHeader_2.54mm:PinHeader_1x05_P2.54mm_Vertical
- removed J6: Sunton P2 IO, Connector_Molex:Molex_PicoBlade_53261-0471_1x04-1MP_P1.25mm_Horizontal
- removed R5, R6, R7: 1k, Resistor_SMD:R_0603_1608Metric
Routing:
- net /IO12_PRESENCE: track 40.1 -> 0.00 mm, vias 6 -> 0
- net /IO13_RXD: track 34.9 -> 0.00 mm, vias 2 -> 0
- net /IO11_TXD: track 29.5 -> 0.00 mm, vias 2 -> 0
- net /+5V: track 108.3 -> 89.0 mm
- net /RADAR_OUT: track 6.51 -> 0.00 mm, vias 1 -> 0
- net /RADAR_TX: track 5.73 -> 0.00 mm
- net /RADAR_RX: track 4.24 -> 0.00 mm
- net /LED_3V3: track 34.3 -> 30.1 mm
- net /SCAN_RX: track 55.3 -> 53.0 mm, vias 4 -> 5
- net /SCAN_TX: track 55.8 -> 56.5 mm, vias 3 -> 0
- net /+3V3: track 21.0 -> 20.3 mm
- net /SCAN_TRIG: vias 0 -> 1
- net /SCAN_STAT: vias 0 -> 1
Other:
- board text removed: "IO11"
- board text removed: "IO12"
- board text removed: "IO13"
- board text removed: "IO19"
- board text removed: "OUT"
- board text removed: "P2 IO"
