File: hardware/scanner-carrier/scanner-carrier.kicad_sch (KiCad schematic)
At the start: 31 parts, among them J1 Sunton P1 UART, J2 Sunton P4 IO, J3 SparkFun 2D Barcode Scanner, J4 GM65 scanner, J5 LD2410C radar, J6 Sunton P2 IO, Q1 AO3400A, U1 AMS1117-3.3, U2 74AHCT1G125

Commit message: Scanner carrier: fix overlapping parts, share the feedback package
The KiCad project defaults came from a demo that ignores courtyard overlaps,
so DRC never checked them. With the check on, six pairs overlapped: the
buzzer, radar header, LED, a corner hole and a test pad are moved apart, and
the second SparkFun standoff (H2) is gone: its hole is 4 mm from the
header's GND pin, so a standoff can't sit next to the socket there. DRC is
clean again with the check on.

Firmware: the buzzer, status LED, presence sensor and the scan feedback
script move to pantry-feedback.yaml, which takes its pins as vars, so the
carrier and the new mainboard share it. The carrier package keeps its radar
UART. The LED uses channel_colors (rgb_order is deprecated).
Parts:
- removed H2: M3 standoff (scanner), MountingHole:MountingHole_3.2mm_M3, symbol Mechanical:MountingHole
Other:
- note added: "SparkFun 2D Barcode Scanner Breakout (DE2120, red aiming line). Plugs in on top; M3 x 11 mm standoff in H1. GM65 instead: J4. Fit only one scanner."
- note removed: "SparkFun 2D Barcode Scanner Breakout (DE2120, red aiming line). Plugs in on top; M3 x 11 mm standoffs in H1/H2. GM65 instead: J4. Fit only one scanner."

Commit message: Drop the presence radar
A scan already wakes the screen, so the LD2410C radar only saved a glance at
the dim clock. Gone from:

- firmware: pantry-feedback.yaml no longer has the presence sensor; the
  carrier package loses the radar UART and ld2410
- scanner carrier: the 5-pin radar header, its three resistors and the
  Sunton P2 connector it needed (two cables to the Sunton now, not three)
- mainboard: the radar header and its resistor; IO4 is free
- enclosure: the radar rails; the chin shrinks to 15 mm, so the case is
  now 111 x 139 x 51 mm

Both boards rebuilt clean (ERC 0, DRC 0 / 0 unconnected / 0 footprint
errors). On the mainboard the ribbon connector is now the only part whose
fine-pitch ground pins rely on the pour; U5's narrow ground pin gets a via
again. All four firmware configs validate.
Parts:
- removed J5: LD2410C radar, Connector_PinHeader_2.54mm:PinHeader_1x05_P2.54mm_Vertical, symbol Connector_Generic:Conn_01x05
- removed J6: Sunton P2 IO, Connector_Molex:Molex_PicoBlade_53261-0471_1x04-1MP_P1.25mm_Horizontal, symbol Connector_Generic:Conn_01x04
- removed R5, R6, R7: 1k, Resistor_SMD:R_0603_1608Metric, symbol Device:R
Connections:
- no-connect marks 2 -> 1
Other:
- note removed: "Radar: HLK-LD2410C on a Dupont cable. OUT -> IO12, UART on IO13 (RX) / IO11 (TX), 256000 baud. IO11-13 are the Sunton SD pins: leave the SD slot empty."
